Commit message: Changed laser scan merger to ira_laser_tools ROS 2 version, added map files of the testing area via SLAM toolbox.

File: hamal_description/urdf/hamal.urdf.xacro (robot description, xacro)
@@ -101,6 +101,11 @@
     <parent link="base_link" />
     <child link="front_scan_link" />
+    <origin xyz="0.91972 0.4838 0.0884" rpy="3.141592 0 0.7853981634" />
+  </joint>
+<!--   <joint name="front_scan_joint" type="fixed">
+    <parent link="base_link" />
+    <child link="front_scan_link" />
     <origin xyz="0.80612 0.3712 0.185" rpy="3.141592 0 0.7853981634" />
-  </joint>
+  </joint> -->
   <link name="front_scan_link">
     <visual>
@@ -121,6 +126,11 @@
     <parent link="base_link" />
     <child link="rear_scan_link" />
+    <origin xyz="-0.91972 -0.4838 0.0884" rpy="3.141592 0  3.926990817 " />
+  </joint>
+<!--   <joint name="rear_scan_joint" type="fixed">
+    <parent link="base_link" />
+    <child link="rear_scan_link" />
     <origin xyz="-0.80612 -0.3712 0.185" rpy="3.141592 0  3.926990817 " />
-  </joint>
+  </joint> -->
   <link name="rear_scan_link">
     <visual>

File: hamal_description/urdf/ros2_control.xacro (robot description, xacro)
@@ -67,5 +67,5 @@
           <param name="position">2</param>
           <param name="mode_of_operation">9</param>
-          <param name="slave_config">$(find hamal_hardware)/config/icube_config.yaml</param>
+          <param name="slave_config">$(find hamal_hardware)/config/left_motor_config.yaml</param>
         </ec_module>
       </joint>
